File: KiCAD/PCB/YM60JIS_PCB.kicad_pcb (KiCad board)
At the start: 2 copper layers, 285.1 x 94.6 mm, 173 parts, among them J1 TYPE-C-31-M-12, SW1 SW_Push, SW10 SW_Push, SW11 SW_Push, SW12 SW_Push, SW13 SW_Push, SW14 SW_Push, SW15 SW_Push, SW16 SW_Push, SW17 SW_Push, SW18 SW_Push, SW19 SW_Push, SW2 SW_Push, SW20 SW_Push, SW21 SW_Push, SW22 SW_Push, SW23 SW_Push, SW24 SW_Push, SW25 SW_Push, SW26 SW_Push, SW27 SW_Push, SW28 SW_Push, SW29 Space, SW3 SW_Push, SW30 SW_Push, SW31 SW_Push, SW32 SW_Push, SW33 SW_Push, SW34 SW_Push, SW35 SW_Push, SW36 SW_Push, SW37 SW_Push, SW38 SW_Push, SW39 SW_Push, SW4 SW_Push, SW40 SW_Push, SW41 SW_Push, SW42 SW_Push, SW43 SW_Push, SW44 SW_Push, SW45 SW_Push, SW46 SW_Push, SW47 SW_Push, SW48 SW_Push, SW49 SW_Push, SW5 SW_Push, SW50 SW_Push, SW51 SW_Push, SW52 SW_Push, SW53 SW_Push, SW54 SW_Push, SW55 SW_Push, SW56 SW_Push, SW57 SW_Push, SW58 SW_Push, SW59 SW_Push, SW6 SW_Push, SW60 SW_Push, SW61 SW_Push, SW62 SW_Push, SW63 Yen, SW64 Backspace, SW65 ISOEnter, SW66 SW_Push, SW67 SW_Push, SW7 SW_Push, SW8 SW_Push, SW9 SW_Push, U1 XC6206P332MR, U2 SMF05CT1G, U3 RP2040, U4 W25Q16JVUXIQ, Y1 X322512MSB4SI

Commit message: Rework PCB and plate for the HHKB-style bottom row (v1.1.2)
- Schematic: switch footprints for the former 1.25u/1.5u bottom-row keys
  are now 1u.
- PCB: move all bottom-row switches and diodes to the new 2.5u-spacebar
  layout, add SW68/D68 (COL4) and SW69/D69 (COL7), replace the 2.75u/3u
  spacebar stabilizers with a 2u stabilizer, and reroute row 4. Move a
  GND via off the new stabilizer hole and the text logo off the かな
  switch. DRC: 0 unconnected pads, no new errors vs v1.1.1.
- Plate: switch and stabilizer cutouts for the new bottom row.
- Version label: "YM60JIS Trilingual v1.1.2 @ymkn & @themrsung".
- PCB and plate are now saved in KiCAD 10 format.
- Add before/after 3D render comparison page (doc/pcb-compare).

Co-Authored-By: Claude Opus 5.5 (1M context) <noreply@anthropic.com>
Parts:
- removed the REF** at (223.8, 133.3) (x2)
- added D68: 1N4148W, Diode_SMD:D_SOD-123, B.Cu at (185.7, 138.1)
- added D69: 1N4148W, Diode_SMD:D_SOD-123, B.Cu at (252.4, 138.1)
- added REF**: STAB_MX_2u, PCM_marbastlib-mx:STAB_MX_2u, F.Cu at (219.1, 133.3)
- added SW68: SW_Push, PCM_marbastlib-mx:SW_MX_HS_CPG151101S11_1u, B.Cu at (185.7, 133.3)
- added SW69: SW_Push, PCM_marbastlib-mx:SW_MX_HS_CPG151101S11_1u, B.Cu at (252.4, 133.3)
- SW10, SW15, SW20, SW47, SW52: footprint PCM_marbastlib-mx:SW_MX_HS_CPG151101S11_1.25u -> PCM_marbastlib-mx:SW_MX_HS_CPG151101S11_1u
- SW5: footprint PCM_marbastlib-mx:SW_MX_HS_CPG151101S11_1.5u -> PCM_marbastlib-mx:SW_MX_HS_CPG151101S11_1u
- moved D20 16.7 mm to (166.7, 138.1)
- moved SW20 16.7 mm to (166.7, 133.3)
- moved D15 11.9 mm to (147.6, 138.1)
- moved SW15 11.9 mm to (147.6, 133.3)
- moved D10 7.14 mm to (128.6, 138.1)
- moved SW10 7.14 mm to (128.6, 133.3)
- moved D42 7.14 mm to (271.5, 138.1)
- moved SW42 7.14 mm to (271.5, 133.3)
- moved G*** 6.05 mm to (236.0, 132.5)
- moved D29 4.76 mm to (219.1, 138.1)
- moved SW29 4.76 mm to (219.1, 133.3)
- moved D5 4.76 mm to (104.8, 138.1)
- moved SW5 4.76 mm to (104.8, 133.3)
- moved D52 2.38 mm to (309.6, 138.1)
- moved SW52 2.38 mm to (309.6, 133.3)
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Routing:
- net COL4: track 138.2 -> 163.1 mm
- net COL7: track 195.2 -> 216.2 mm
- net ROW4: track 380.0 -> 399.9 mm, vias 12 -> 14
- net Net-(D69-A): track 0.00 -> 11.6 mm
- net Net-(D68-A): track 0.00 -> 11.6 mm
- net COL2: track 107.3 -> 112.2 mm
- net COL3: track 139.2 -> 144.1 mm
- net COL8: track 238.1 -> 235.1 mm
- net COL1: track 147.0 -> 150.0 mm
- net COL0: track 103.3 -> 105.3 mm
- net COL5: track 178.2 -> 176.2 mm
- net COL9: track 255.7 -> 254.7 mm
- net COL10: track 273.1 -> 274.1 mm
Other:
- board text added: "YM60JIS Trilingual v1.1.2 @ymkn & @themrsung"
- board text removed: "YM60JIS v1.1.1 @ymkn"
