File: KiCAD/PCB/YM60JIS_PCB.kicad_sch (KiCad schematic)
At the start: 165 parts, among them J1 TYPE-C-31-M-12, SW1 SW_Push, SW10 SW_Push, SW11 SW_Push, SW12 SW_Push, SW13 SW_Push, SW14 SW_Push, SW15 SW_Push, SW16 SW_Push, SW17 SW_Push, SW18 SW_Push, SW19 SW_Push, SW2 SW_Push, SW20 SW_Push, SW21 SW_Push, SW22 SW_Push, SW23 SW_Push, SW24 SW_Push, SW25 SW_Push, SW26 SW_Push, SW27 SW_Push, SW28 SW_Push, SW29 Space, SW3 SW_Push, SW30 SW_Push, SW31 SW_Push, SW32 SW_Push, SW33 SW_Push, SW34 SW_Push, SW35 SW_Push, SW36 SW_Push, SW37 SW_Push, SW38 SW_Push, SW39 SW_Push, SW4 SW_Push, SW40 SW_Push, SW41 SW_Push, SW42 SW_Push, SW43 SW_Push, SW44 SW_Push, SW45 SW_Push, SW46 SW_Push, SW47 SW_Push, SW48 SW_Push, SW49 SW_Push, SW5 SW_Push, SW50 SW_Push, SW51 SW_Push, SW52 SW_Push, SW53 SW_Push, SW54 SW_Push, SW55 SW_Push, SW56 SW_Push, SW57 SW_Push, SW58 SW_Push, SW59 SW_Push, SW6 SW_Push, SW60 SW_Push, SW61 SW_Push, SW62 SW_Push, SW63 Yen, SW64 Backspace, SW65 ISOEnter, SW66 SW_Push, SW67 SW_Push, SW7 SW_Push, SW8 SW_Push, SW9 SW_Push, U1 XC6206P332MR, U2 SMF05CT1G, U3 RP2040, U4 W25Q16JVUXIQ, Y1 X322512MSB4SI

Commit message: Trilingual fork initial commit
Rework the bottom row into an HHKB-style macOS layout:
Fn, Lang3, Option, Command, 英数, Space (2.5u), かな, Command, Option, Fn,
with 0.25u gaps before Lang3 and before the arrow keys.

- Firmware: new row 4 layout using matrix (4,4) and (4,7); HHKB mapping
  with Control on Caps and the HHKB Fn layer; Lang3 sends KC_GRV.
  Fix row 3 x offsets in keyboard.json.
- Vial: update the bottom row definition.
- Schematic: add SW68/D68 (COL4) and SW69/D69 (COL7) on ROW4.
- Docs: rewrite README and build guide in English for the new layout;
  add base and Fn layer diagrams.

PCB and plate are not yet updated.

Co-Authored-By: Claude Opus 5.5 (1M context) <noreply@anthropic.com>
Parts:
- added D68, D69: 1N4148W, Diode_SMD:D_SOD-123, symbol Diode:1N4148W
- added SW68, SW69: SW_Push, PCM_marbastlib-mx:SW_MX_HS_CPG151101S11_1u, symbol Switch:SW_Push
Connections:
- net COL4: now also SW68.1
- net COL7: now also SW69.1
- net ROW4: now also D68.1 (K), D69.1 (K)
- new net: D69.2 (A), SW69.2
- new net: D68.2 (A), SW68.2

Commit message: Rework PCB and plate for the HHKB-style bottom row (v1.1.2)
- Schematic: switch footprints for the former 1.25u/1.5u bottom-row keys
  are now 1u.
- PCB: move all bottom-row switches and diodes to the new 2.5u-spacebar
  layout, add SW68/D68 (COL4) and SW69/D69 (COL7), replace the 2.75u/3u
  spacebar stabilizers with a 2u stabilizer, and reroute row 4. Move a
  GND via off the new stabilizer hole and the text logo off the かな
  switch. DRC: 0 unconnected pads, no new errors vs v1.1.1.
- Plate: switch and stabilizer cutouts for the new bottom row.
- Version label: "YM60JIS Trilingual v1.1.2 @ymkn & @themrsung".
- PCB and plate are now saved in KiCAD 10 format.
- Add before/after 3D render comparison page (doc/pcb-compare).

Co-Authored-By: Claude Opus 5.5 (1M context) <noreply@anthropic.com>
Parts:
- SW10, SW15, SW20, SW47, SW52: footprint PCM_marbastlib-mx:SW_MX_HS_CPG151101S11_1.25u -> PCM_marbastlib-mx:SW_MX_HS_CPG151101S11_1u
- SW5: footprint PCM_marbastlib-mx:SW_MX_HS_CPG151101S11_1.5u -> PCM_marbastlib-mx:SW_MX_HS_CPG151101S11_1u
Changed lines of the file:
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@@
 			)
 		)
-		(property "Footprint" "PCM_marbastlib-mx:SW_MX_HS_CPG151101S11_1.25u"
+		(property "Footprint" "PCM_marbastlib-mx:SW_MX_HS_CPG151101S11_1u"
 			(at 265.43 102.87 0)
 			(effects
@@
 			)
 		)
-		(property "Footprint" "PCM_marbastlib-mx:SW_MX_HS_CPG151101S11_1.25u"
+		(property "Footprint" "PCM_marbastlib-mx:SW_MX_HS_CPG151101S11_1u"
 			(at 59.69 102.87 0)
 			(effects
@@
 			)
 		)
-		(property "Footprint" "PCM_marbastlib-mx:SW_MX_HS_CPG151101S11_1.25u"
+		(property "Footprint" "PCM_marbastlib-mx:SW_MX_HS_CPG151101S11_1u"
 			(at 105.41 102.87 0)
 			(effects
@@
 			)
 		)
-		(property "Footprint" "PCM_marbastlib-mx:SW_MX_HS_CPG151101S11_1.25u"
+		(property "Footprint" "PCM_marbastlib-mx:SW_MX_HS_CPG151101S11_1u"
 			(at 82.55 102.87 0)
 			(effects
@@
 			)
 		)
-		(property "Footprint" "PCM_marbastlib-mx:SW_MX_HS_CPG151101S11_1.5u"
+		(property "Footprint" "PCM_marbastlib-mx:SW_MX_HS_CPG151101S11_1u"
 			(at 36.83 102.87 0)
 			(effects
@@
 			)
 		)
-		(property "Footprint" "PCM_marbastlib-mx:SW_MX_HS_CPG151101S11_1.25u"
+		(property "Footprint" "PCM_marbastlib-mx:SW_MX_HS_CPG151101S11_1u"
 			(at 242.57 102.87 0)
 			(effects
